Commit message: completed core drone model, added inertial macros, saved rviz2 drone frame viewer

File: ros2_ws/src/drone/description/robot_core.xacro (robot description, xacro)
@@ -1,4 +1,6 @@
 <?xml version="1.0"?>
 <robot xmlns:xacro="http://www.ros.org/wiki/xacro">
+    <!-- Include inertia macros -->
+    <xacro:include filename="inertia_macros.xacro"/>
     <!--  COMMONLY USED COLORS -->
     <material name="white">
@@ -16,11 +18,27 @@
     <!-- BASE LINK -->
     <link name="base_link">
-        <visual>
-            <geometry>
-                <box size="0.5 0.3 0.3"/>
+    </link>
+    <!-- FRAME -->
+    <joint name="frame_joint" type="fixed">
+        <parent link="base_link"/>
+        <child link="frame_link"/>
+        <origin xyz = "0 0 0.024"/>
+    </joint>
+    <link name="frame_link">
+        <visual>
+            <geometry>
+                <box size="0.13 0.045 0.02"/>
             </geometry>
             <material name="white"/>
-            <origin xyz="0 0 0" rpy="0 0 0" /> <!-- At center of frame -->
-        </visual>
+            <origin xyz="0 0 -0.01" rpy="0 0 0" />
+        </visual>
+        <collision>
+            <geometry>
+                <box size="0.13 0.045 0.02"/>
+            </geometry>
+            <origin xyz="0 0 -0.01" rpy="0 0 0" />
+        </collision>
+        <!-- inertia -->
+        <xacro:box mass="0.306" x="0.13" y="0.045" z="0.02" origin_xyz="0 0 -0.01" origin_rpy="0 0 0"/>
     </link>
     <!-- FRONT LEFT MOTOR ARM -->
@@ -28,14 +46,22 @@
         <parent link="base_link"/>
         <child link="fl_motor"/>
-        <origin xyz="0.707 0.707 0" rpy="0 0 0"/>
+        <origin xyz="0.0707 0.0707 0" rpy="0 0 ${-pi/4 - pi/2}"/>
     </joint>
     <link name="fl_motor">
         <visual>
             <geometry>
-                <cylinder length="1" radius="0.1"/>
-            </geometry>
-            <material name="orange"/>
-            <origin xyz="-0.3535 -0.3535 0" rpy= "0 1.57 0.785"/>
-        </visual>
+                <cylinder length="0.1" radius="0.004"/>
+            </geometry>
+            <material name="orange"/>
+            <origin xyz="0.05 0 0" rpy= "0 1.57 0"/>
+        </visual>
+        <collision>
+            <geometry>
+                <cylinder length="0.1" radius="0.004"/>
+            </geometry>
+            <origin xyz="0.05 0 0" rpy= "0 1.57 0"/>
+        </collision>
+        <!-- inertia -->
+        <xacro:cyl_end_x mass="0.016" r="0.004" l="0.1" origin_xyz="0.0211 0 0" origin_rpy="0 0 0"/>
     </link>
     <!-- FRONT RIGHT MOTOR ARM -->
@@ -43,14 +69,22 @@
         <parent link="base_link"/>
         <child link="fr_motor"/>
-        <origin xyz="0.707 -0.707 0" rpy="0 0 0" />
+        <origin xyz="0.0707 -0.0707 0" rpy="0 0 ${pi/4 + pi/2}" />
     </joint>
     <link name="fr_motor">
         <visual>
             <geometry>
-                <cylinder length="1" radius="0.1"/>
-            </geometry>
-            <material name="orange"/>
-            <origin xyz="-0.3535 0.3535 0" rpy= "0 1.57 -0.785"/>
-        </visual>
+                <cylinder length="0.1" radius="0.004"/>
+            </geometry>
+            <material name="orange"/>
+            <origin xyz="0.05 0 0" rpy= "0 1.57 0"/>
+        </visual>
+        <collision>
+            <geometry>
+                <cylinder length="0.1" radius="0.004"/>
+            </geometry>
+            <origin xyz="0.05 0 0" rpy= "0 1.57 0"/>
+        </collision>
+        <!-- inertia -->
+        <xacro:cyl_end_x mass="0.016" r="0.004" l="0.1" origin_xyz="0.0211 0 0" origin_rpy="0 0 0"/>
     </link>
     <!-- BACK LEFT MOTOR ARM -->
@@ -58,14 +92,22 @@
         <parent link="base_link"/>
         <child link="bl_motor"/>
-        <origin xyz="-0.707 0.707 0" rpy="0 0 0" />
+        <origin xyz="-0.0707 0.0707 0" rpy="0 0 ${-pi/4}" />
     </joint>
     <link name="bl_motor">
         <visual>
             <geometry>
-                <cylinder length="1" radius="0.1"/>
-            </geometry>
-            <material name="orange"/>
-            <origin xyz="0.3535 -0.3535 0" rpy= "0 1.57 -0.785"/>
-        </visual>
+                <cylinder length="0.1" radius="0.004"/>
+            </geometry>
+            <material name="orange"/>
+            <origin xyz="0.05 0 0" rpy= "0 1.57 0"/>
+        </visual>
+        <collision>
+            <geometry>
+                <cylinder length="0.1" radius="0.004"/>
+            </geometry>
+            <origin xyz="0.05 0.05 0" rpy= "0 1.57 0"/>
+        </collision>
+        <!-- inertia -->
+        <xacro:cyl_end_x mass="0.016" r="0.004" l="0.1" origin_xyz="0.0211 0 0" origin_rpy="0 0 0"/>
     </link>
     <!-- BACK RIGHT MOTOR ARM -->
@@ -73,14 +115,22 @@
         <parent link="base_link"/>
         <child link="br_motor"/>
-        <origin xyz="-0.707 -0.707 0" rpy="0 0 0" />
+        <origin xyz="-0.0707 -0.0707 0" rpy="0 0 ${pi/4}" />
     </joint>
     <link name="br_motor">
         <visual>
             <geometry>
-                <cylinder length="1" radius="0.1"/>
-            </geometry>
-            <material name="orange"/>
-            <origin xyz="0.3535 0.3535 0" rpy= "0 1.57 0.785"/>
-        </visual>
+                <cylinder length="0.1" radius="0.004"/>
+            </geometry>
+            <material name="orange"/>
+            <origin xyz="0.05 0 0" rpy= "0 1.57 0"/>
+        </visual>
+        <collision>
+            <geometry>
+                <cylinder length="0.1" radius="0.004"/>
+            </geometry>
+            <origin xyz="0.05 0 0" rpy= "0 1.57 0"/>
+        </collision>
+        <!-- inertia -->
+        <xacro:cyl_end_x mass="0.016" r="0.004" l="0.1" origin_xyz="0.0211 0 0" origin_rpy="0 0 0"/>
     </link>
     <!-- FRONT LEFT PROPELLER -->
@@ -88,13 +138,23 @@
         <parent link="fl_motor"/>
         <child link="fl_prop"/>
-        <origin xyz="0 0 0.1" rpy="0 0 0"/>
+        <origin xyz="0 0 0.01" rpy="0 0 0"/>
+        <axis xyz="0 0 1"/>
     </joint>
     <link name="fl_prop">
         <visual>
             <geometry>
-                <cylinder length="0.004" radius="0.0635"/>
-            </geometry>
-            <material name="blue"/>
-        </visual>
+                <cylinder length="0.004" radius="0.038"/>
+            </geometry>
+            <material name="blue"/>
+            <origin xyz="0 0 0"/>
+        </visual>
+        <collision>
+            <geometry>
+                <cylinder length="0.004" radius="0.038"/>
+            </geometry>
+            <origin xyz="0 0 0"/>
+        </collision>
+        <!-- inertia -->
+        <xacro:cyl_center_z mass="0.003" r="0.038" l="0.004"/>
     </link>
     <!-- FRONT RIGHT PROPELLER -->
@@ -102,14 +162,23 @@
         <parent link="fr_motor"/>
         <child link="fr_prop"/>
-        <origin xyz="0 0 0.1" rpy="0 0 0"/>
+        <origin xyz="0 0 0.01" rpy="0 0 0"/>
+        <axis xyz="0 0 -1"/>
     </joint>
     <link name="fr_prop">
         <visual>
             <geometry>
-                <cylinder length="0.004" radius="0.0635"/>
-            </geometry>
-            <material name="blue"/>
-            <origin xyz="0 0 0"/>
-        </visual>
+                <cylinder length="0.004" radius="0.038"/>
+            </geometry>
+            <material name="blue"/>
+            <origin xyz="0 0 0"/>
+        </visual>
+        <collision>
+            <geometry>
+                <cylinder length="0.004" radius="0.038"/>
+            </geometry>
+            <origin xyz="0 0 0"/>
+        </collision>
+        <!-- inertia -->
+        <xacro:cyl_center_z mass="0.003" r="0.038" l="0.004"/>
     </link>
     <!-- BACK LEFT PROPELLER -->
@@ -117,14 +186,23 @@
         <parent link="bl_motor"/>
         <child link="bl_prop"/>
-        <origin xyz="0 0 0.1" rpy="0 0 0"/>
+        <origin xyz="0 0 0.01" rpy="0 0 0"/>
+        <axis xyz="0 0 -1"/>
     </joint>
     <link name="bl_prop">
         <visual>
             <geometry>
-                <cylinder length="0.004" radius="0.0635"/>
-            </geometry>
-            <material name="blue"/>
-            <origin xyz="0 0 0"/>
-        </visual>
+                <cylinder length="0.004" radius="0.038"/>
+            </geometry>
+            <material name="blue"/>
+            <origin xyz="0 0 0"/>
+        </visual>
+        <collision>
+            <geometry>
+                <cylinder length="0.004" radius="0.038"/>
+            </geometry>
+            <origin xyz="0 0 0"/>
+        </collision>
+        <!-- inertia -->
+        <xacro:cyl_center_z mass="0.003" r="0.038" l="0.004"/>
     </link>
     <!-- BACK RIGHT PROPELLER -->
@@ -132,14 +210,23 @@
         <parent link="br_motor"/>
         <child link="br_prop"/>
-        <origin xyz="0 0 0.1" rpy="0 0 0"/>
+        <origin xyz="0 0 0.01" rpy="0 0 0"/>
+        <axis xyz="0 0 1"/>
     </joint>
     <link name="br_prop">
         <visual>
             <geometry>
-                <cylinder length="0.004" radius="0.0635"/>
-            </geometry>
-            <material name="blue"/>
-            <origin xyz="0 0 0"/>
-        </visual>
+                <cylinder length="0.004" radius="0.038"/>
+            </geometry>
+            <material name="blue"/>
+            <origin xyz="0 0 0"/>
+        </visual>
+        <collision>
+            <geometry>
+                <cylinder length="0.004" radius="0.038"/>
+            </geometry>
+            <origin xyz="0 0 0"/>
+        </collision>
+        <!-- inertia -->
+        <xacro:cyl_center_z mass="0.003" r="0.038" l="0.004"/>
     </link>
 </robot>
