Commit message: Created simulated lidar sensor, created test gazebo world for simulation

File: ros2_ws/src/drone/description/robot.urdf.xacro (robot description, xacro)
@@ -3,3 +3,4 @@
     <!-- Base Drone Frame -->
     <xacro:include filename="robot_core.xacro"/>
+    <xacro:include filename="lidar.xacro"/>
 </robot>

File: ros2_ws/src/drone/description/robot_core.xacro (robot description, xacro)
@@ -16,4 +16,7 @@
         <color rgba="0.2 0.2 1 1" />
     </material>
+    <material name="red">
+        <color rgba="1 0 0 1" />
+    </material>
     <!-- BASE LINK -->
     <link name="base_link">
@@ -42,4 +45,7 @@
         <xacro:box mass="0.306" x="0.13" y="0.045" z="0.02" origin_xyz="0 0 -0.01" origin_rpy="0 0 0"/>
     </link>
+    <gazebo reference="frame_link">
+        <material>Gazebo/White</material>
+    </gazebo>
     <!-- FRONT LEFT MOTOR ARM -->
     <joint name="fl_motor_joint" type="fixed">
@@ -65,4 +71,7 @@
         <xacro:cyl_end_x mass="0.016" r="0.004" l="0.1" origin_xyz="0.0211 0 0" origin_rpy="0 0 0"/>
     </link>
+    <gazebo reference="fl_motor">
+        <material>Gazebo/Orange</material>
+    </gazebo>
     <!-- FRONT RIGHT MOTOR ARM -->
     <joint name="fr_motor_joint" type="fixed">
@@ -88,4 +97,7 @@
         <xacro:cyl_end_x mass="0.016" r="0.004" l="0.1" origin_xyz="0.0211 0 0" origin_rpy="0 0 0"/>
     </link>
+    <gazebo reference="fr_motor">
+        <material>Gazebo/Orange</material>
+    </gazebo>
     <!-- BACK LEFT MOTOR ARM -->
     <joint name="bl_motor_joint" type="fixed">
@@ -111,4 +123,7 @@
         <xacro:cyl_end_x mass="0.016" r="0.004" l="0.1" origin_xyz="0.0211 0 0" origin_rpy="0 0 0"/>
     </link>
+    <gazebo reference="bl_motor">
+        <material>Gazebo/Orange</material>
+    </gazebo>
     <!-- BACK RIGHT MOTOR ARM -->
     <joint name="br_motor_joint" type="fixed">
@@ -134,4 +149,7 @@
         <xacro:cyl_end_x mass="0.016" r="0.004" l="0.1" origin_xyz="0.0211 0 0" origin_rpy="0 0 0"/>
     </link>
+    <gazebo reference="br_motor">
+        <material>Gazebo/Orange</material>
+    </gazebo>
     <!-- FRONT LEFT PROPELLER -->
     <joint name="fl_prop_joint" type="continuous">
@@ -146,16 +164,19 @@
                 <cylinder length="0.004" radius="0.038"/>
             </geometry>
-            <material name="blue"/>
-            <origin xyz="0 0 0"/>
-        </visual>
-        <collision>
-            <geometry>
-                <cylinder length="0.004" radius="0.038"/>
-            </geometry>
-            <origin xyz="0 0 0"/>
-        </collision>
-        <!-- inertia -->
-        <xacro:cyl_center_z mass="0.003" r="0.038" l="0.004"/>
-    </link>
+            <material name="black"/>
+            <origin xyz="0 0 0"/>
+        </visual>
+        <collision>
+            <geometry>
+                <cylinder length="0.004" radius="0.038"/>
+            </geometry>
+            <origin xyz="0 0 0"/>
+        </collision>
+        <!-- inertia -->
+        <xacro:cyl_center_z mass="0.003" r="0.038" l="0.004"/>
+    </link>
+    <gazebo reference="fl_prop">
+        <material>Gazebo/Black</material>
+    </gazebo>
     <!-- FRONT RIGHT PROPELLER -->
      <joint name="fr_prop_joint" type="continuous">
@@ -170,16 +191,19 @@
                 <cylinder length="0.004" radius="0.038"/>
             </geometry>
-            <material name="blue"/>
-            <origin xyz="0 0 0"/>
-        </visual>
-        <collision>
-            <geometry>
-                <cylinder length="0.004" radius="0.038"/>
-            </geometry>
-            <origin xyz="0 0 0"/>
-        </collision>
-        <!-- inertia -->
-        <xacro:cyl_center_z mass="0.003" r="0.038" l="0.004"/>
-    </link>
+            <material name="black"/>
+            <origin xyz="0 0 0"/>
+        </visual>
+        <collision>
+            <geometry>
+                <cylinder length="0.004" radius="0.038"/>
+            </geometry>
+            <origin xyz="0 0 0"/>
+        </collision>
+        <!-- inertia -->
+        <xacro:cyl_center_z mass="0.003" r="0.038" l="0.004"/>
+    </link>
+    <gazebo reference="fr_prop">
+        <material>Gazebo/Black</material>
+    </gazebo>
     <!-- BACK LEFT PROPELLER -->
      <joint name="bl_prop_joint" type="continuous">
@@ -194,16 +218,19 @@
                 <cylinder length="0.004" radius="0.038"/>
             </geometry>
-            <material name="blue"/>
-            <origin xyz="0 0 0"/>
-        </visual>
-        <collision>
-            <geometry>
-                <cylinder length="0.004" radius="0.038"/>
-            </geometry>
-            <origin xyz="0 0 0"/>
-        </collision>
-        <!-- inertia -->
-        <xacro:cyl_center_z mass="0.003" r="0.038" l="0.004"/>
-    </link>
+            <material name="black"/>
+            <origin xyz="0 0 0"/>
+        </visual>
+        <collision>
+            <geometry>
+                <cylinder length="0.004" radius="0.038"/>
+            </geometry>
+            <origin xyz="0 0 0"/>
+        </collision>
+        <!-- inertia -->
+        <xacro:cyl_center_z mass="0.003" r="0.038" l="0.004"/>
+    </link>
+    <gazebo reference="bl_prop">
+        <material>Gazebo/Black</material>
+    </gazebo>
     <!-- BACK RIGHT PROPELLER -->
      <joint name="br_prop_joint" type="continuous">
@@ -218,15 +245,18 @@
                 <cylinder length="0.004" radius="0.038"/>
             </geometry>
-            <material name="blue"/>
-            <origin xyz="0 0 0"/>
-        </visual>
-        <collision>
-            <geometry>
-                <cylinder length="0.004" radius="0.038"/>
-            </geometry>
-            <origin xyz="0 0 0"/>
-        </collision>
-        <!-- inertia -->
-        <xacro:cyl_center_z mass="0.003" r="0.038" l="0.004"/>
-    </link>
+            <material name="black"/>
+            <origin xyz="0 0 0"/>
+        </visual>
+        <collision>
+            <geometry>
+                <cylinder length="0.004" radius="0.038"/>
+            </geometry>
+            <origin xyz="0 0 0"/>
+        </collision>
+        <!-- inertia -->
+        <xacro:cyl_center_z mass="0.003" r="0.038" l="0.004"/>
+    </link>
+    <gazebo reference="br_prop">
+        <material>Gazebo/Black</material>
+    </gazebo>
 </robot>
